File: pcb/ControlPanel.kicad_pcb (KiCad board)
At the start: 4 copper layers, 120 x 75 mm, 325 parts, among them IC1 NS2009, IC2 TPS61240DRVT, IC3 ATA6561-GAQW-N, IC4 MAX2674EWT+T, J1 MCSP-Q-08-A-SG-T_R, J10 Conn_01x02, J11 TC2030, J12 Conn_01x07_Socket, J13 Conn_01x05_Socket, J14 Conn_01x08_Socket, J15 Conn_01x12_Socket, J16 Conn_01x01, J17 Conn_01x01, J19 Conn_01x01, J2 MEM2067-02-180-00-A, J20 Conn_01x01, J3 BATT, J4 Conn_01x02, J5 Conn_01x02, J7 Conn_Coaxial_Small, J8 Conn_Coaxial_Small, J9 TF07V-40S-0.5SH_800_, Q2 BSS138, T1 H1102NL, U1 MCP2518FD-xQBB, U10 USBLC6-2SC6, U11 TPA6132A2RTE, U2 V3S, U3 TPS54360DDA, U4 SY8088AAC, U5 STM32L432KCUx, U6 MAX-M10S, U7 AXP209, U701 GAQY212GS, U702 GAQY212GS, U8 TPS61041DBV, U9 USBLC6-2SC6, Y1 3225-20M-SR, Y2 CX2016FB24000D0FZZ, Y3 32.768kHz

Commit message: Cleaning
Parts:
- U2: footprint FunKey:ELQFP-128 -> Local_L:ELQFP-128
- U4: footprint FunKey:SOT23-5 -> Package_TO_SOT_SMD:SOT-23-5
- U7: footprint AXP209_QFN48:AXP209-QFN48 -> Local_L:AXP209-QFN48
- turned U4 to 90 degrees
