File: pcb/ControlPanel.kicad_pcb (KiCad board)
At the start: 4 copper layers, 120 x 75 mm, 325 parts, among them IC1 NS2009, IC2 TPS61240DRVT, IC3 ATA6561-GAQW-N, IC4 MAX2674EWT+T, J1 MCSP-Q-08-A-SG-T_R, J10 Conn_01x02, J11 TC2030, J12 Conn_01x07_Socket, J13 Conn_01x05_Socket, J14 Conn_01x08_Socket, J15 Conn_01x12_Socket, J16 Conn_01x01, J17 Conn_01x01, J19 Conn_01x01, J2 MEM2067-02-180-00-A, J20 Conn_01x01, J3 BATT, J4 Conn_01x02, J5 Conn_01x02, J7 Conn_Coaxial_Small, J8 Conn_Coaxial_Small, J9 TF07V-40S-0.5SH_800_, Q2 BSS138, T1 H1102NL, U1 MCP2518FD-xQBB, U10 USBLC6-2SC6, U11 TPA6132A2RTE, U2 V3S, U3 TPS54360DDA, U4 SY8088AAC, U5 STM32L432KCUx, U6 MAX-M10S, U7 AXP209, U701 GAQY212GS, U702 GAQY212GS, U8 TPS61041DBV, U9 USBLC6-2SC6, Y1 3225-20M-SR, Y2 CX2016FB24000D0FZZ, Y3 32.768kHz

Commit message: Unify values/footprints per checklist, add via-in-pad DRC rule, regenerate outputs
Parts:
- C52: footprint Capacitor_SMD:C_1206_3216Metric_Pad1.33x1.80mm_HandSolder -> Capacitor_SMD:C_1206_3216Metric
- R29, R3, R4: value 200k 1% -> 200k
- moved TP11 3.13 mm to (125.7, 89.3)
- moved C44 0.15 mm to (113.2, 80.6)
Routing:
- net /AUDIO/G1: track 67.4 -> 84.6 mm, vias 2 -> 5
- net GND: track 119.7 -> 130.3 mm, vias 2809 -> 2767
- net +3V3_AO: track 87.8 -> 92.7 mm
- net +3V3_PWR: track 247.6 -> 248.9 mm, vias 14 -> 18
- net /CPU/I2C_SCL: track 145.1 -> 146.1 mm
- net /AUDIO/EN: track 59.0 -> 59.9 mm, vias 2 -> 4
- net /CPU/I2C_SDA: track 144.8 -> 145.5 mm
- net /AUDIO/G0: track 63.9 -> 64.0 mm, vias 2 -> 4
- net /CPU_PWR/DC_IN: vias 28 -> 26

Commit message: Final fixes
Parts:
- added FID1: Fiducial, Fiducial:Fiducial_0.5mm_Mask1mm, F.Cu at (91.0, 67.6)
- added FID2: Fiducial, Fiducial:Fiducial_0.5mm_Mask1mm, F.Cu at (181.0, 109.5)
Routing:
- net +3V3_PWR: track 248.9 -> 249.8 mm
- net /AUDIO/EN: track 59.9 -> 60.6 mm
- net /AUDIO/G0: track 64.0 -> 64.6 mm
- net GND: vias 2767 -> 2762
