File: pcb/audio.kicad_sch (KiCad schematic)
At the start: 28 parts, among them J14 Conn_01x08_Socket, U11 TPA6132A2RTE

Commit message: Fix BOM data: correct MPN for 33R resistors (R52/R55/R56), BOM export settings
Parts:
- R46, R47: Manufacturer_Part_Number ERJ3EKF1623V -> (none)
