File: pcb/cpu.kicad_sch (KiCad schematic)
At the start: 64 parts, among them J10 Conn_01x02, U2 V3S, Y2 CX2016FB24000D0FZZ, Y3 32.768kHz

Commit message: Cleaning
Parts:
- U2: footprint FunKey:ELQFP-128 -> Local_L:ELQFP-128
Changed lines of the file:
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@@
 			)
 		)
-		(property "Footprint" "FunKey:ELQFP-128"
+		(property "Footprint" "Local_L:ELQFP-128"
 			(at 153.67 157.48 0)
 			(hide yes)
@@
 			(at 153.67 157.48 0)
 			(hide yes)
-			(show_name no)
-			(do_not_autoplace no)
-			(effects
-				(font
-					(size 1.27 1.27)
-				)
-			)
-		)
-		(property "MPN" ""
-			(at 153.67 157.48 0)
-			(hide yes)
-			(show_name no)
-			(do_not_autoplace no)
-			(effects
-				(font
-					(size 1.27 1.27)
-				)
-			)
-		)
-		(property "PARTNO" ""
-			(at 153.67 157.48 0)
-			(hide yes)

Commit message: Unify values/footprints per checklist, add via-in-pad DRC rule, regenerate outputs
Parts:
- R29, R3: value 200k 1% -> 200k
Changed lines of the file:
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@@
 			)
 		)
-		(property "Value" "200k 1%"
+		(property "Value" "200k"
 			(at 161.29 59.6899 0)
 			(show_name no)
@@
 			)
 		)
-		(property "Value" "200k 1%"
+		(property "Value" "200k"
 			(at 363.22 118.1099 0)
 			(show_name no)

Commit message: Fix BOM data: correct MPN for 33R resistors (R52/R55/R56), BOM export settings
Parts:
- R52: Manufacturer_Part_Number ERJ3EKF1623V -> (none)
