File: pcb/cpu_pwr.kicad_sch (KiCad schematic)
At the start: 49 parts, among them J3 BATT, J4 Conn_01x02, J5 Conn_01x02, U7 AXP209

Commit message: Cleaning
Parts:
- U7: footprint AXP209_QFN48:AXP209-QFN48 -> Local_L:AXP209-QFN48; LCSC C2997895 -> (none)
Changed lines of the file:
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@@
 		(fields_autoplaced yes)
 		(property "Reference" "U7"
-			(at 132.08 21.59 0)
+			(at 132.08 20.32 0)
 			(show_name no)
 			(do_not_autoplace no)
@@
 		)
 		(property "Value" "AXP209"
-			(at 132.08 24.13 0)
+			(at 132.08 22.86 0)
 			(show_name no)
 			(do_not_autoplace no)
@@
 			)
 		)
-		(property "Footprint" "AXP209_QFN48:AXP209-QFN48"
+		(property "Footprint" "Local_L:AXP209-QFN48"
 			(at 134.62 151.13 0)
 			(hide yes)
@@
 			(show_name no)
 			(do_not_autoplace no)
-			(effects
-				(font
-					(size 1.27 1.27)
-				)
-			)
-		)
-		(property "LCSC" "C2997895"
-			(at 137.16 73.66 0)
-			(hide yes)
-			(show_name no)
-			(do_not_autoplace no)
-			(effects
-				(font
-					(size 1.27 1.27)
-				)
-			)
-		)
-		(property "PARTNO" ""
-			(at 137.16 73.66 0)
-			(hide yes)
-			(show_name no)
-			(do_not_autoplace no)

Commit message: Unify values/footprints per checklist, add via-in-pad DRC rule, regenerate outputs
Parts:
- R4: value 200k 1% -> 200k
Changed lines of the file:
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@@
 			)
 		)
-		(property "Value" "200k 1%"
+		(property "Value" "200k"
 			(at 174.498 127.4322 0)
 			(show_name no)

Commit message: Final fixes
Changed lines of the file:
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@@
 		(dnp no)
 		(property "Reference" "C10"
-			(at 90.17 76.2 90)
+			(at 91.186 76.2 90)
 			(show_name no)
 			(do_not_autoplace no)
