File: pcb/eth.kicad_sch (KiCad schematic)
At the start: 20 parts, among them T1 H1102NL, U10 USBLC6-2SC6, U9 USBLC6-2SC6

Commit message: Unify values/footprints per checklist, add via-in-pad DRC rule, regenerate outputs
Parts:
- C52: footprint Capacitor_SMD:C_1206_3216Metric_Pad1.33x1.80mm_HandSolder -> Capacitor_SMD:C_1206_3216Metric
Changed lines of the file:
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@@
 			)
 		)
-		(property "Footprint" "Capacitor_SMD:C_1206_3216Metric_Pad1.33x1.80mm_HandSolder"
+		(property "Footprint" "Capacitor_SMD:C_1206_3216Metric"
 			(at 182.5752 125.73 0)
 			(hide yes)
