File: pcb/memory.kicad_sch (KiCad schematic)
At the start: 22 parts, among them J1 MCSP-Q-08-A-SG-T_R, J2 MEM2067-02-180-00-A

Commit message: Fix BOM data: correct MPN for 33R resistors (R52/R55/R56), BOM export settings
Parts:
- R55, R56: Manufacturer_Part_Number ERJ3EKF1623V -> (none)
